File: HM-LC-SW1-BA-PCB_mini_MAX1724-Kicad/HM-LC-SW1-BA-PCB_mini_MAX1724.sch (KiCad schematic (older format))
At the start: 28 parts, among them IC1 ATMEGA328P-A, IC2 CC1101, J1 Conn_01x03_Female, J2 Conn_01x03_Female, P3 ANT, P4 ISP Bottom, P5 ISP Top, Q1 TSM2302, SW1 Reset, SW2 Config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

Commit message: update to V0.3
improvement GND area inductor
Other:
- note added: "ANT: 72mm Wire"
Changed lines of the file:
@@
 EESchema Schematic File Version 4
-EELAYER 29 0
+LIBS:HM-LC-SW1-BA-PCB_mini_MAX1724-cache
+EELAYER 30 0
 EELAYER END
 $Descr A4 11693 8268
@@
 Title "HM-LC-SW1-BA-PCB_mini_MAX1724"
 Date ""
-Rev "0.2"
+Rev "0.3"
 Comp ""
-Comment1 "V0.2"
+Comment1 "V0.3"
 Comment2 ""
 Comment3 ""
@@
 Wire Notes Line
 	1275 2875 1275 1525
+Text Notes 9975 2200 0    79   ~ 16
+ANT: 72mm Wire
 $EndSCHEMATC
