File: HM-LC-SW1-BA-PCB_mini_MAX1724-Kicad/HM-LC-SW1-BA-PCB_mini_MAX1724.kicad_pcb (KiCad board)
At the start: 2 copper layers, 20 x 40 mm, 28 parts, among them IC1 ATMEGA328P-A, IC2 CC1101, J1 Conn_01x02_Female, J2 Conn_01x03_Female, P3 ANT, P4 ISP Bottom, P5 ISP Top, Q1 TSM2302, SW1 Reset, SW2 Config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

Commit message: update to V0.2
Parts:
- removed TP1: TestPoint, TestPoint:TestPoint_Pad_D1.0mm
- added C4: 9p, Capacitor_SMD:C_0805_2012Metric_Pad1.15x1.40mm_HandSolder, F.Cu at (186.8, 96.9)
- added C5: 9p, Capacitor_SMD:C_0805_2012Metric_Pad1.15x1.40mm_HandSolder, F.Cu at (180.8, 94.8)
- added Y1: Crystal, Crystal:Crystal_SMD_MicroCrystal_CC7V-T1A-2Pin_3.2x1.5mm_HandSoldering, F.Cu at (181.4, 97.2)
- C1, C2, C3, C6, C7: footprint Capacitors_SMD:C_0805_HandSoldering -> Capacitor_SMD:C_0805_2012Metric_Pad1.15x1.40mm_HandSolder
- J1: value Conn_01x02_Female -> Conn_01x03_Female; footprint Connector_PinHeader_2.54mm:PinHeader_1x02_P2.54mm_Vertical -> Connector_PinHeader_2.54mm:PinHeader_1x03_P2.54mm_Vertical
- Q1: value TSM2302 -> IRLML2803
- moved R3 2.62 mm to (180.8, 92.4)
- moved Q1 2.15 mm to (176.7, 91.6)
- moved R6 2.12 mm to (180.8, 90.3)
- moved R2 2.10 mm to (186.5, 92.2), turned to 0 degrees
- moved C1 1.13 mm to (186.9, 100.2)
- moved C2 0.42 mm to (175.9, 109.5)
- moved C3 0.38 mm to (187.6, 110.0)
- moved L1 0.30 mm to (183.7, 118.3)
- moved C7 0.16 mm to (178.3, 121.2)
Connections:
- IC1 pad 10: /RELAY -> Net-(IC1-Pad10)
- IC1 pad 9: Net-(IC1-Pad9) -> /RELAY
Routing:
- net Net-(IC1-Pad2): track 9.48 -> 17.4 mm
- net /XTAL2: track 0.00 -> 6.40 mm
- net /RELAY: track 7.09 -> 11.1 mm
- net /XTAL1: track 4.08 -> 6.98 mm
- net /OUTPUT: track 22.0 -> 24.5 mm
- net Net-(Q1-Pad1): track 4.75 -> 7.11 mm
- net VCC: track 126.7 -> 124.4 mm
- net /A0: track 34.5 -> 32.9 mm, vias 6 -> 4
- net Net-(D1-Pad2): track 3.69 -> 2.25 mm
- net GND: track 20.0 -> 20.2 mm, vias 27 -> 21
Other:
- board text added: "CC BY-SA-NC 4.0"
- board text added: "HM-LC-SW1-BA-PCB_mini StepUp/ext. Batt meas. V0.2"
- board text removed: "CC BY-NC-SA 4.0"
- board text removed: "HM-LC-SW1-BA-PCB_mini StepUp/ext. Batt meas. V0.1"
- board text removed: "XTAL1"

Commit message: update V0.2
Parts:
- moved C6 0.90 mm to (177.5, 115.2)
- moved C7 0.85 mm to (178.3, 122.0), turned to 180 degrees
- moved L1 0.61 mm to (183.1, 118.2), turned to 90 degrees
- moved U1 0.36 mm to (178.4, 118.5), turned to 90 degrees
Routing:
- net Net-(L1-Pad2): track 7.65 -> 4.14 mm
- net VCC: track 124.4 -> 121.4 mm, vias 4 -> 3
- net GND: track 20.2 -> 17.9 mm
- net /A0: track 32.9 -> 34.5 mm
- net /Vin: track 32.6 -> 33.3 mm

Commit message: update V0.2
Routing:
- net /A0: track 34.5 -> 36.7 mm
Changed lines of the file:
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@@
     (thickness 1.6)
     (drawings 23)
-    (tracks 440)
+    (tracks 442)
     (zones 0)
     (modules 30)
@@
   (gr_line (start 190 85) (end 190 125) (angle 90) (layer Edge.Cuts) (width 0.15))
   (gr_line (start 170 85) (end 190 85) (angle 90) (layer Edge.Cuts) (width 0.15))
-  (via (at 186.75 107.9) (size 0.6) (drill 0.4) (layers F.Cu B.Cu) (net 2))
-  (via (at 181.8 120.5) (size 0.6) (drill 0.4) (layers F.Cu B.Cu) (net 22))
   (segment (start 189.23 88.9762) (end 189.23 92.5068) (width 0.25) (layer B.Cu) (net 1))
   (segment (start 189.23 95.061738) (end 189.23 94.6404) (width 0.25) (layer B.Cu) (net 1))
@@
   (segment (start 180.875736 113.7864) (end 180.489336 113.4) (width 0.25) (layer B.Cu) (net 1))
   (segment (start 181.3 113.7864) (end 180.875736 113.7864) (width 0.25) (layer B.Cu) (net 1))
+  (segment (start 177.45 116.275) (end 178.525 115.2) (width 0.5) (layer B.Cu) (net 1))
+  (segment (start 177.45 117.24) (end 177.45 116.275) (width 0.5) (layer B.Cu) (net 1))
+  (segment (start 178.025 113.9) (end 177.9 113.9) (width 0.5) (layer B.Cu) (net 1))
+  (segment (start 178.525 114.4) (end 178.025 113.9) (width 0.5) (layer B.Cu) (net 1))
+  (segment (start 178.525 115.2) (end 178.525 114.4) (width 0.5) (layer B.Cu) (net 1))
+  (segment (start 178.7 113.9) (end 177.9 113.9) (width 0.5) (layer B.Cu) (net 1))
+  (segment (start 177.9 113.9) (end 177 113.9) (width 0.5) (layer B.Cu) (net 1))
+  (via (at 186.75 107.9) (size 0.6) (drill 0.4) (layers F.Cu B.Cu) (net 2))
   (via (at 176.5 110.6) (size 0.6) (drill 0.4) (layers F.Cu B.Cu) (net 2))
   (via (at 178.7 88.2) (size 0.6) (drill 0.4) (layers F.Cu B.Cu) (net 2))
@@
   (via (at 188.225 102.45) (size 0.6) (drill 0.4) (layers F.Cu B.Cu) (net 2))
   (via (at 188.2 103.8) (size 0.6) (drill 0.4) (layers F.Cu B.Cu) (net 2))
-  (segment (start 177.45 116.275) (end 178.525 115.2) (width 0.5) (layer B.Cu) (net 1))
-  (segment (start 177.45 117.24) (end 177.45 116.275) (width 0.5) (layer B.Cu) (net 1))
-  (segment (start 178.025 113.9) (end 177.9 113.9) (width 0.5) (layer B.Cu) (net 1))
-  (segment (start 178.525 114.4) (end 178.025 113.9) (width 0.5) (layer B.Cu) (net 1))
-  (segment (start 178.525 115.2) (end 178.525 114.4) (width 0.5) (layer B.Cu) (net 1))
-  (segment (start 178.7 113.9) (end 177.9 113.9) (width 0.5) (layer B.Cu) (net 1))
-  (segment (start 177.9 113.9) (end 177 113.9) (width 0.5) (layer B.Cu) (net 1))
   (segment (start 186.699027 102.1334) (end 185.711917 103.12051) (width 0.25) (layer F.Cu) (net 3))
   (via (at 186.6 102.25) (size 0.6) (drill 0.4) (layers F.Cu B.Cu) (net 3))
@@
   (segment (start 179.70151 109.130917) (end 177.933614 110.898813) (width 0.25) (layer F.Cu) (net 15))
   (via (at 174.4 116.2) (size 0.6) (drill 0.4) (layers F.Cu B.Cu) (net 15))
-  (via (at 174.4 118.525) (size 0.6) (drill 0.4) (layers F.Cu B.Cu) (net 15))
+  (via (at 174.4 118.25) (size 0.6) (drill 0.4) (layers F.Cu B.Cu) (net 15))
   (segment (start 176.932427 111.9) (end 177.933614 110.898813) (width 0.25) (layer F.Cu) (net 15))
   (segment (start 175.8 111.9) (end 176.932427 111.9) (width 0.25) (layer F.Cu) (net 15))
@@
   (segment (start 175.1 115.5) (end 174.4 116.2) (width 0.25) (layer B.Cu) (net 15))
   (segment (start 175.1 114.85) (end 175.1 115.5) (width 0.25) (layer B.Cu) (net 15))
-  (segment (start 174.4 118.525) (end 174.4 116.2) (width 0.25) (layer F.Cu) (net 15))
-  (segment (start 174.4 120.975) (end 174.4 118.525) (width 0.25) (layer B.Cu) (net 15))
   (segment (start 176.725 123.3) (end 174.4 120.975) (width 0.25) (layer B.Cu) (net 15))
   (segment (start 180 123.35) (end 181.05 123.35) (width 0.25) (layer B.Cu) (net 15))
@@
   (segment (start 181.05 123.35) (end 185.95 123.35) (width 0.25) (layer F.Cu) (net 15))
   (segment (start 188.6585 120.6415) (end 188.6585 118.6815) (width 0.25) (layer F.Cu) (net 15))
+  (segment (start 174.4 116.2) (end 174.4 118.25) (width 0.25) (layer F.Cu) (net 15))
+  (segment (start 174.4 118.25) (end 174.4 120.8) (width 0.25) (layer B.Cu) (net 15))
+  (segment (start 174.4 120.975) (end 174.4 120.8) (width 0.25) (layer B.Cu) (net 15))
+  (segment (start 174.4 120.8) (end 174.4 118.525) (width 0.25) (layer B.Cu) (net 15))
   (segment (start 179.578 113.5215) (end 176.6151 113.5215) (width 0.25) (layer F.Cu) (net 17))
   (segment (start 176.6151 113.5215) (end 176.6062 113.5304) (width 0.25) (layer F.Cu) (net 17))
@@
   (segment (start 179.825 95.1) (end 179.475 94.75) (width 0.25) (layer F.Cu) (net 19))
   (segment (start 179.825 97.1) (end 179.825 95.1) (width 0.25) (layer F.Cu) (net 19))
+  (via (at 181.8 120.5) (size 0.6) (drill 0.4) (layers F.Cu B.Cu) (net 22))
   (segment (start 184.5 113.05) (end 184.75 112.8) (width 0.25) (layer B.Cu) (net 22))
   (segment (start 179.6565 116.3) (end 179.578 116.2215) (width 0.25) (layer F.Cu) (net 22))

Commit message: update to V0.3
improvement GND area inductor
Other:
- board text added: "ANT: 72mm Wire"
- board text added: "HM-LC-SW1-BA-PCB_mini StepUp/ext. Batt meas."
- board text added: "V0.3"
- board text removed: "HM-LC-SW1-BA-PCB_mini StepUp/ext. Batt meas. V0.2"
Changed lines of the file:
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@@
-(kicad_pcb (version 20171130) (host pcbnew "(5.1.2)-2")
+(kicad_pcb (version 20171130) (host pcbnew "(5.1.4)-1")
   (general
     (thickness 1.6)
-    (drawings 23)
+    (drawings 25)
     (tracks 442)
     (zones 0)
@@
     )
   )
+  (gr_text "ANT: 72mm Wire" (at 180.68 90.65) (layer B.SilkS)
+    (effects (font (size 0.8 0.8) (thickness 0.15)) (justify mirror))
+  )
+  (gr_text V0.3 (at 189.04 109.78 90) (layer F.SilkS)
+    (effects (font (size 0.8 0.8) (thickness 0.15)))
+  )
   (gr_text "CC BY-SA-NC 4.0" (at 179.85 123.85) (layer F.SilkS)
     (effects (font (size 0.8 0.8) (thickness 0.15)))
@@
     (effects (font (size 1 1) (thickness 0.2)))
   )
-  (gr_text "HM-LC-SW1-BA-PCB_mini\nStepUp/ext. Batt meas.\nV0.2" (at 172.35 106.6 90) (layer F.SilkS)
+  (gr_text "HM-LC-SW1-BA-PCB_mini\nStepUp/ext. Batt meas." (at 171.86 106.64 90) (layer F.SilkS)
     (effects (font (size 0.6 0.55) (thickness 0.1)))
   )
@@
       )
     )
+  )
+  (zone (net 0) (net_name "") (layer F.Cu) (hatch edge 0.508)
+    (connect_pads (clearance 0.4))
+    (min_thickness 0.254)
+    (keepout (tracks allowed) (vias allowed) (copperpour not_allowed))
+    (fill (arc_segments 32) (thermal_gap 0.508) (thermal_bridge_width 0.508))
+    (polygon
+      (pts
+        (xy 181.13987 115.98) (xy 180.6 115.98) (xy 180.6125 114.585) (xy 184.45 114.53) (xy 185.06 115.2)
+        (xy 184.992115 121.940021) (xy 184.8 122.16) (xy 181.340048 122.141196) (xy 181.13 121.87)
+      )
+    )

Commit message: V0.3
some small fixes
Routing:
- net /Vin: track 33.3 -> 34.4 mm
Changed lines of the file:
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@@
     (thickness 1.6)
     (drawings 25)
-    (tracks 442)
+    (tracks 444)
     (zones 0)
     (modules 30)
@@
   )
   (setup
-    (last_trace_width 0.25)
+    (last_trace_width 0.5)
     (user_trace_width 0.5)
     (user_trace_width 1)
@@
     (uvia_drill 0.1)
   )
+  (module Package_TO_SOT_SMD:SOT-23 (layer F.Cu)
+    (at 176.7 91.6 270)
+    (descr "SOT-23, Standard")
+    (tags SOT-23)
+    (attr smd)
+    (fp_text reference Q1 (at 1.4 1.4 180) (layer F.SilkS)
+      (effects (font (size 0.8 0.8) (thickness 0.15)))
+    )
+    (fp_text value IRLML2803 (at 0 2.5 270) (layer F.Fab)
+      (effects (font (size 1 1) (thickness 0.15)))
+    )
+    (fp_line (start 0.76 1.58) (end -0.7 1.58) (layer F.SilkS) (width 0.12))
+    (fp_line (start 0.76 -1.58) (end -1.4 -1.58) (layer F.SilkS) (width 0.12))
+    (fp_line (start -1.7 1.75) (end -1.7 -1.75) (layer F.CrtYd) (width 0.05))
+    (fp_line (start 1.7 1.75) (end -1.7 1.75) (layer F.CrtYd) (width 0.05))
+    (fp_line (start 1.7 -1.75) (end 1.7 1.75) (layer F.CrtYd) (width 0.05))
+    (fp_line (start -1.7 -1.75) (end 1.7 -1.75) (layer F.CrtYd) (width 0.05))
+    (fp_line (start 0.76 -1.58) (end 0.76 -0.65) (layer F.SilkS) (width 0.12))
+    (fp_line (start 0.76 1.58) (end 0.76 0.65) (layer F.SilkS) (width 0.12))
+    (fp_line (start -0.7 1.52) (end 0.7 1.52) (layer F.Fab) (width 0.1))
+    (fp_line (start 0.7 -1.52) (end 0.7 1.52) (layer F.Fab) (width 0.1))
+    (fp_line (start -0.7 -0.95) (end -0.15 -1.52) (layer F.Fab) (width 0.1))
+    (fp_line (start -0.15 -1.52) (end 0.7 -1.52) (layer F.Fab) (width 0.1))
+    (fp_line (start -0.7 -0.95) (end -0.7 1.5) (layer F.Fab) (width 0.1))
+    (fp_text user %R (at 0 0) (layer F.Fab)
+      (effects (font (size 0.5 0.5) (thickness 0.075)))
+    )
+    (pad 3 smd rect (at 1.175 0 270) (size 1.2 0.8) (layers F.Cu F.Paste F.Mask)
+      (net 25 /OUTPUT))
+    (pad 2 smd rect (at -1.15 0.95 270) (size 1.2 0.8) (layers F.Cu F.Paste F.Mask)
+      (net 2 GND))
+    (pad 1 smd rect (at -1.15 -0.95 270) (size 1.2 0.8) (layers F.Cu F.Paste F.Mask)
+      (net 26 "Net-(Q1-Pad1)"))
+    (model ${KISYS3DMOD}/Package_TO_SOT_SMD.3dshapes/SOT-23.wrl
+      (at (xyz 0 0 0))
+      (scale (xyz 1 1 1))
+      (rotate (xyz 0 0 0))
+    )
+  )
   (module Connector_PinHeader_2.54mm:PinHeader_1x03_P2.54mm_Vertical (layer F.Cu)
     (at 171.3 113.6)
@@
       (net 26 "Net-(Q1-Pad1)"))
     (model ${KISYS3DMOD}/Resistor_SMD.3dshapes/R_0805_2012Metric.wrl
-      (at (xyz 0 0 0))
-      (scale (xyz 1 1 1))
-      (rotate (xyz 0 0 0))
-    )
-  )
-  (module Package_TO_SOT_SMD:SOT-23 (layer F.Cu)
-    (at 176.7 91.6 270)
-    (descr "SOT-23, Standard")
-    (tags SOT-23)
-    (attr smd)
-    (fp_text reference Q1 (at 1.4 1.4 180) (layer F.SilkS)
-      (effects (font (size 0.8 0.8) (thickness 0.15)))
-    )
-    (fp_text value IRLML2803 (at 0 2.5 90) (layer F.Fab)
-      (effects (font (size 1 1) (thickness 0.15)))
-    )
-    (fp_line (start 0.76 1.58) (end -0.7 1.58) (layer F.SilkS) (width 0.12))
-    (fp_line (start 0.76 -1.58) (end -1.4 -1.58) (layer F.SilkS) (width 0.12))
-    (fp_line (start -1.7 1.75) (end -1.7 -1.75) (layer F.CrtYd) (width 0.05))
-    (fp_line (start 1.7 1.75) (end -1.7 1.75) (layer F.CrtYd) (width 0.05))
-    (fp_line (start 1.7 -1.75) (end 1.7 1.75) (layer F.CrtYd) (width 0.05))
-    (fp_line (start -1.7 -1.75) (end 1.7 -1.75) (layer F.CrtYd) (width 0.05))
-    (fp_line (start 0.76 -1.58) (end 0.76 -0.65) (layer F.SilkS) (width 0.12))
-    (fp_line (start 0.76 1.58) (end 0.76 0.65) (layer F.SilkS) (width 0.12))
-    (fp_line (start -0.7 1.52) (end 0.7 1.52) (layer F.Fab) (width 0.1))
-    (fp_line (start 0.7 -1.52) (end 0.7 1.52) (layer F.Fab) (width 0.1))
-    (fp_line (start -0.7 -0.95) (end -0.15 -1.52) (layer F.Fab) (width 0.1))
-    (fp_line (start -0.15 -1.52) (end 0.7 -1.52) (layer F.Fab) (width 0.1))
-    (fp_line (start -0.7 -0.95) (end -0.7 1.5) (layer F.Fab) (width 0.1))
-    (fp_text user %R (at 0 0) (layer F.Fab)
-      (effects (font (size 0.5 0.5) (thickness 0.075)))
-    )
-    (pad 3 smd rect (at 1 0 270) (size 0.9 0.8) (layers F.Cu F.Paste F.Mask)
-      (net 25 /OUTPUT))
-    (pad 2 smd rect (at -1 0.95 270) (size 0.9 0.8) (layers F.Cu F.Paste F.Mask)
-      (net 2 GND))
-    (pad 1 smd rect (at -1 -0.95 270) (size 0.9 0.8) (layers F.Cu F.Paste F.Mask)
-      (net 26 "Net-(Q1-Pad1)"))
-    (model ${KISYS3DMOD}/Package_TO_SOT_SMD.3dshapes/SOT-23.wrl
       (at (xyz 0 0 0))
       (scale (xyz 1 1 1))
@@
   (segment (start 188.6585 113.6015) (end 187.707 112.65) (width 0.5) (layer B.Cu) (net 22))
   (segment (start 187.707 112.65) (end 184.75 112.65) (width 0.5) (layer B.Cu) (net 22))
-  (segment (start 188.6585 113.6015) (end 185.9985 113.6015) (width 0.5) (layer B.Cu) (net 22))
-  (segment (start 185.25001 118.84999) (end 184.975 119.125) (width 0.5) (layer B.Cu) (net 22))
-  (segment (start 185.25001 114.34999) (end 185.25001 118.84999) (width 0.5) (layer B.Cu) (net 22))
-  (segment (start 185.9985 113.6015) (end 185.25001 114.34999) (width 0.5) (layer B.Cu) (net 22))
-  (segment (start 184.975 119.125) (end 183.1 121) (width 0.5) (layer B.Cu) (net 22))
   (segment (start 182.02929 119.92929) (end 180.12071 119.92929) (width 0.5) (layer B.Cu) (net 22))
   (segment (start 183.1 121) (end 182.02929 119.92929) (width 0.5) (layer B.Cu) (net 22))
@@
   (segment (start 180.5 116.2215) (end 181.8 117.5215) (width 0.25) (layer F.Cu) (net 22))
   (segment (start 179.6 116.2215) (end 180.5 116.2215) (width 0.25) (layer F.Cu) (net 22))
+  (segment (start 184.96 121) (end 183.1 121) (width 0.5) (layer B.Cu) (net 22))
+  (segment (start 185.9985 113.6015) (end 185.25001 114.34999) (width 0.5) (layer B.Cu) (net 22))
+  (segment (start 188.6585 113.6015) (end 185.9985 113.6015) (width 0.5) (layer B.Cu) (net 22))
+  (segment (start 185.25001 114.34999) (end 185.25001 118.84999) (width 0.5) (layer B.Cu) (net 22))
+  (segment (start 185.25001 118.84999) (end 185.25 118.85) (width 0.5) (layer B.Cu) (net 22))
+  (segment (start 185.25 118.85) (end 185.25 120.71) (width 0.5) (layer B.Cu) (net 22))
+  (segment (start 185.25 120.71) (end 184.96 121) (width 0.5) (layer B.Cu) (net 22))
   (segment (start 179.807225 101.529169) (end 179.807225 101.63538) (width 0.25) (layer F.Cu) (net 23))
   (segment (start 179.135824 100.857768) (end 179.807225 101.529169) (width 0.25) (layer F.Cu) (net 23))

Commit message: V0.3
some small fixes
Parts:
- moved L1 0.57 mm to (183.1, 117.6)
Routing:
- net /RESET: track 38.5 -> 40.9 mm
- net VCC: track 121.4 -> 119.6 mm
- net /Vin: track 34.4 -> 35.3 mm
